File: pocket_mixer.sch (KiCad schematic (older format))
At the start: 41 parts, among them J1 PJ3410, J2 PJ3410, U1 4580, U2 4580, U3 4580, U4 4580

Commit message: update to kicad version 5, bug fix layout
Parts:
- C1, C11, C12, C13, C14, C2, C3, C4, C47, C48, C5, C6, C7, C8: symbol C -> pocket_mixer-rescue:C
- C10, C15, C16, C9: symbol CP -> pocket_mixer-rescue:CP
- J1, J2: symbol PJ3410 -> pocket_mixer-rescue:PJ3410
- R1, R10, R11, R12, R13, R14, R15, R16, R2, R3, R4, R5, R6, R7, R8, R9: symbol R -> pocket_mixer-rescue:R
- RV1: symbol POT_Dual -> pocket_mixer-rescue:POT_Dual
- U1, U2, U3, U4: symbol 4558 -> pocket_mixer-rescue:4558
