File: vu_meter.sch (KiCad schematic (older format))
At the start: 11 parts, among them U13 LM3914

Commit message: update to kicad version 5, bug fix layout
Parts:
- D10, D11, D12, D13, D14, D5, D6, D7, D8, D9: symbol LED -> pocket_mixer-rescue:LED
- U13: symbol LM3914 -> pocket_mixer-rescue:LM3914
Changed lines of the file:
@@
-EESchema Schematic File Version 2
-LIBS:power
-LIBS:device
-LIBS:transistors
-LIBS:conn
-LIBS:linear
-LIBS:regul
-LIBS:74xx
-LIBS:cmos4000
-LIBS:adc-dac
-LIBS:memory
-LIBS:xilinx
-LIBS:microcontrollers
-LIBS:dsp
-LIBS:microchip
-LIBS:analog_switches
-LIBS:motorola
-LIBS:texas
-LIBS:intel
-LIBS:audio
-LIBS:interface
-LIBS:digital-audio
-LIBS:philips
-LIBS:display
-LIBS:cypress
-LIBS:siliconi
-LIBS:opto
-LIBS:atmel
-LIBS:contrib
-LIBS:valves
-LIBS:switches
-LIBS:stahllabs
+EESchema Schematic File Version 4
 LIBS:pocket_mixer-cache
-EELAYER 25 0
+EELAYER 26 0
 EELAYER END
 $Descr A4 11693 8268
@@
 $EndDescr
 $Comp
-L LM3914 U13
+L pocket_mixer-rescue:LM3914 U13
 U 1 1 5966459C
 P 5650 3950
@@
 $EndComp
 $Comp
-L +12V #PWR0112
+L pocket_mixer-rescue:+12V #PWR0112
 U 1 1 59664BB1
 P 5650 3150
@@
 $EndComp
 $Comp
-L +12V #PWR0113
+L pocket_mixer-rescue:+12V #PWR0113
 U 1 1 59664FF6
 P 4800 4100
@@
 $EndComp
 $Comp
-L LED D5
+L pocket_mixer-rescue:LED D5
 U 1 1 59665099
 P 6700 2550
@@
 $EndComp
 $Comp
-L LED D6
+L pocket_mixer-rescue:LED D6
 U 1 1 596650CE
 P 6700 2850
@@
 $EndComp
 $Comp
-L LED D7
+L pocket_mixer-rescue:LED D7
 U 1 1 596650F9
 P 6700 3150
@@
 $EndComp
 $Comp
-L LED D8
+L pocket_mixer-rescue:LED D8
 U 1 1 59665121
 P 6700 3450
@@
 $EndComp
 $Comp
-L LED D9
+L pocket_mixer-rescue:LED D9
 U 1 1 5966514C
 P 6700 3750
@@
 $EndComp
 $Comp
-L LED D10
+L pocket_mixer-rescue:LED D10
 U 1 1 5966517E
 P 6700 4050
@@
 $EndComp
 $Comp
-L LED D11
+L pocket_mixer-rescue:LED D11
 U 1 1 596651AF
 P 6700 4350
@@
 $EndComp
 $Comp
-L LED D12
+L pocket_mixer-rescue:LED D12
 U 1 1 596651DF
 P 6700 4650
@@
 $EndComp
 $Comp
-L LED D13
+L pocket_mixer-rescue:LED D13
 U 1 1 5966521F
 P 6700 4950
@@
 $EndComp
 $Comp
-L LED D14
+L pocket_mixer-rescue:LED D14
 U 1 1 59665255
 P 6700 5250
@@
 Connection ~ 6850 2850
 $Comp
-L +12V #PWR0114
+L pocket_mixer-rescue:+12V #PWR0114
 U 1 1 59665859
 P 6850 2350
