File: inputs_1-3.sch (KiCad schematic (older format))
At the start: 45 parts, among them J3 PJ3410, J4 PJ3410, J5 PJ3410, U5 4580, U6 4580, U7 4580

Commit message: update to kicad version 5, bug fix layout
Parts:
- C17, C18, C19, C20, C29, C30: symbol CP -> pocket_mixer-rescue:CP
- C21, C22, C23, C24, C25, C26, C27, C28, C31, C32, C33, C34: symbol C -> pocket_mixer-rescue:C
- J3, J4, J5: symbol PJ3410 -> pocket_mixer-rescue:PJ3410
- R17, R18, R19, R20, R21, R22, R23, R24, R25, R26, R27, R28, R29, R30, R31, R32, R33, R34: symbol R -> pocket_mixer-rescue:R
- RV2, RV3, RV4: symbol POT_Dual -> pocket_mixer-rescue:POT_Dual
- U5, U6, U7: symbol 4558 -> pocket_mixer-rescue:4558
Connections:
- wire segments 110 -> 138

Commit message: :rocket: 2.0.0
Parts:
- added JP? (x3): SolderJumper_2_Open, symbol Jumper:SolderJumper_2_Open
- added unit 3 of U5
- added unit 3 of U6
- added unit 3 of U7
- C17, C18, C19, C20, C29, C30: symbol pocket_mixer-rescue:CP -> Device:CP
- C21, C22, C23, C24, C25, C26, C27, C28, C31, C32, C33, C34: symbol pocket_mixer-rescue:C -> Device:C
- J3, J4, J5: symbol pocket_mixer-rescue:PJ3410 -> stahllabs:PJ3410
- R17, R18, R19, R20, R21, R22, R23, R24, R25, R26, R27, R28, R29, R30, R31, R32, R33, R34: symbol pocket_mixer-rescue:R -> Device:R
- RV2, RV3, RV4: symbol pocket_mixer-rescue:POT_Dual -> Device:R_POT_Dual
- U5, U6, U7: value 4580 -> NJM4580; symbol pocket_mixer-rescue:4558 -> Amplifier_Operational:NJM4580
Connections:
- wire segments 138 -> 156
