File: inputs_4_return.sch (KiCad schematic (older format))
At the start: 30 parts, among them J6 PJ3410, J7 PJ3410, U8 4580, U9 4580

Commit message: update to kicad version 5, bug fix layout
Parts:
- C35, C36, C41, C42: symbol CP -> pocket_mixer-rescue:CP
- C37, C38, C39, C40, C43, C44, C45, C46: symbol C -> pocket_mixer-rescue:C
- J6, J7: symbol PJ3410 -> pocket_mixer-rescue:PJ3410
- R53, R54, R55, R56, R57, R58, R59, R60, R61, R62, R63, R64: symbol R -> pocket_mixer-rescue:R
- RV10, RV9: symbol POT_Dual -> pocket_mixer-rescue:POT_Dual
- U8, U9: symbol 4558 -> pocket_mixer-rescue:4558
Changed lines of the file:
@@
-EESchema Schematic File Version 2
-LIBS:power
-LIBS:device
-LIBS:transistors
-LIBS:conn
-LIBS:linear
-LIBS:regul
-LIBS:74xx
-LIBS:cmos4000
-LIBS:adc-dac
-LIBS:memory
-LIBS:xilinx
-LIBS:microcontrollers
-LIBS:dsp
-LIBS:microchip
-LIBS:analog_switches
-LIBS:motorola
-LIBS:texas
-LIBS:intel
-LIBS:audio
-LIBS:interface
-LIBS:digital-audio
-LIBS:philips
-LIBS:display
-LIBS:cypress
-LIBS:siliconi
-LIBS:opto
-LIBS:atmel
-LIBS:contrib
-LIBS:valves
-LIBS:switches
-LIBS:stahllabs
+EESchema Schematic File Version 4
 LIBS:pocket_mixer-cache
-EELAYER 25 0
+EELAYER 26 0
 EELAYER END
 $Descr A4 11693 8268
@@
 4-RIGHT
 $Comp
-L GND #PWR080
+L pocket_mixer-rescue:GND #PWR080
 U 1 1 5928C0B6
 P 1650 2100
@@
 $EndComp
 $Comp
-L GND #PWR081
+L pocket_mixer-rescue:GND #PWR081
 U 1 1 5928C0BC
 P 1650 2600
@@
 LEVEL
 $Comp
-L C C40
+L pocket_mixer-rescue:C C40
 U 1 1 5928C0C3
 P 4650 1350
@@
 $EndComp
 $Comp
-L C C39
+L pocket_mixer-rescue:C C39
 U 1 1 5928C0CA
 P 4300 1350
@@
 $EndComp
 $Comp
-L GND #PWR082
+L pocket_mixer-rescue:GND #PWR082
 U 1 1 5928C0D1
 P 4650 1500
@@
 $EndComp
 $Comp
-L GND #PWR083
+L pocket_mixer-rescue:GND #PWR083
 U 1 1 5928C0D7
 P 4300 1500
@@
 $EndComp
 $Comp
-L POT_Dual RV9
+L pocket_mixer-rescue:POT_Dual RV9
 U 1 1 5928C0E9
 P 1900 2500
@@
 $EndComp
 $Comp
-L R R56
+L pocket_mixer-rescue:R R56
 U 1 1 5928C0FC
 P 3000 3050
@@
 $EndComp
 $Comp
-L R R55
+L pocket_mixer-rescue:R R55
 U 1 1 5928C103
 P 3000 2250
@@
 $EndComp
 $Comp
-L R R54
+L pocket_mixer-rescue:R R54
 U 1 1 5928C116
 P 2950 3950
@@
 $EndComp
 $Comp
-L GND #PWR084
+L pocket_mixer-rescue:GND #PWR084
 U 1 1 5928C11D
 P 2650 1100
@@
 $EndComp
 $Comp
-L R R53
+L pocket_mixer-rescue:R R53
 U 1 1 5928C123
 P 2950 1000
@@
 $EndComp
 $Comp
-L C C38
+L pocket_mixer-rescue:C C38
 U 1 1 5928C12A
 P 3600 3700
@@
 $EndComp
 $Comp
-L C C37
+L pocket_mixer-rescue:C C37
 U 1 1 5928C131
 P 3600 1300
@@
 $EndComp
 $Comp
-L R R58
+L pocket_mixer-rescue:R R58
 U 1 1 5928C138
 P 3600 3950
@@
 $EndComp
 $Comp
-L R R57
+L pocket_mixer-rescue:R R57
 U 1 1 5928C13F
 P 3600 1000
@@
 $EndComp
 $Comp
-L 4558 U8
+L pocket_mixer-rescue:4558 U8
 U 2 1 5928C158
 P 3650 3000
@@
 $EndComp
 $Comp
-L 4558 U8
+L pocket_mixer-rescue:4558 U8
 U 1 1 5928C15F
 P 3650 2000
@@
 	1450 2650 1450 2950
 $Comp
-L GND #PWR085
+L pocket_mixer-rescue:GND #PWR085
 U 1 1 5928C16A
 P 1300 2800
@@
 	1300 2700 1300 2800
 $Comp
-L PJ3410 J6
+L pocket_mixer-rescue:PJ3410 J6
 U 1 1 5928C172
 P 1250 2600
@@
 $EndComp
 $Comp
-L CP C35
+L pocket_mixer-rescue:CP C35
 U 1 1 5928C179
 P 2650 2100
@@
 $EndComp
 $Comp
-L CP C36
+L pocket_mixer-rescue:CP C36
 U 1 1 5928C180
 P 2650 2900
@@
 RETURN-RIGHT
 $Comp
-L GND #PWR086
+L pocket_mixer-rescue:GND #PWR086
 U 1 1 5928D4D4
 P 6400 2100
@@
 $EndComp
 $Comp
-L GND #PWR087
+L pocket_mixer-rescue:GND #PWR087
 U 1 1 5928D4DA
 P 6400 2600
@@
 LEVEL
 $Comp
-L C C46
+L pocket_mixer-rescue:C C46
 U 1 1 5928D4E1
 P 9400 1350
@@
 $EndComp
 $Comp
-L C C45
+L pocket_mixer-rescue:C C45
 U 1 1 5928D4E8
 P 9050 1350
@@
 $EndComp
 $Comp
-L GND #PWR088
+L pocket_mixer-rescue:GND #PWR088
 U 1 1 5928D4EF
 P 9400 1500
@@
 $EndComp
 $Comp
-L GND #PWR089
+L pocket_mixer-rescue:GND #PWR089
 U 1 1 5928D4F5
 P 9050 1500
@@
 $EndComp
 $Comp
-L POT_Dual RV10
+L pocket_mixer-rescue:POT_Dual RV10
 U 1 1 5928D507
 P 6650 2500
@@
 $EndComp
 $Comp
-L GND #PWR090
+L pocket_mixer-rescue:GND #PWR090
 U 1 1 5928D50E
 P 7750 3200
@@
 $EndComp
 $Comp
-L GND #PWR091
+L pocket_mixer-rescue:GND #PWR091
 U 1 1 5928D514
 P 7750 2400
@@
 $EndComp
 $Comp
-L R R62
+L pocket_mixer-rescue:R R62
 U 1 1 5928D51A
 P 7750 3050
@@
 $EndComp
 $Comp
-L R R61
+L pocket_mixer-rescue:R R61
 U 1 1 5928D521
 P 7750 2250
@@
 $EndComp
 $Comp
-L GND #PWR092
+L pocket_mixer-rescue:GND #PWR092
 U 1 1 5928D52E
 P 7400 4050
@@
 $EndComp
 $Comp
-L R R60
+L pocket_mixer-rescue:R R60
 U 1 1 5928D534
 P 7700 3950
@@
 $EndComp
 $Comp
-L GND #PWR093
+L pocket_mixer-rescue:GND #PWR093
 U 1 1 5928D53B
 P 7400 1100
@@
 $EndComp
 $Comp
-L R R59
+L pocket_mixer-rescue:R R59
 U 1 1 5928D541
 P 7700 1000
@@
 $EndComp
 $Comp
-L C C44
+L pocket_mixer-rescue:C C44
 U 1 1 5928D548
 P 8350 3700
@@
 $EndComp
 $Comp
-L C C43
+L pocket_mixer-rescue:C C43
 U 1 1 5928D54F
 P 8350 1300
@@
 $EndComp
 $Comp
-L R R64
+L pocket_mixer-rescue:R R64
 U 1 1 5928D556
 P 8350 3950
@@
 $EndComp
 $Comp
-L R R63
+L pocket_mixer-rescue:R R63
 U 1 1 5928D55D
 P 8350 1000
@@
 $EndComp
 $Comp
-L 4558 U9
+L pocket_mixer-rescue:4558 U9
 U 2 1 5928D576
 P 8400 3000
@@
 $EndComp
 $Comp
-L 4558 U9
+L pocket_mixer-rescue:4558 U9
 U 1 1 5928D57D
 P 8400 2000
@@
 	6200 2650 6200 2950
 $Comp
-L GND #PWR094
+L pocket_mixer-rescue:GND #PWR094
 U 1 1 5928D588
 P 6050 2800
@@
 	6050 2700 6050 2800
 $Comp
-L PJ3410 J7
+L pocket_mixer-rescue:PJ3410 J7
 U 1 1 5928D590
 P 6000 2600
@@
 $EndComp
 $Comp
-L CP C41
+L pocket_mixer-rescue:CP C41
 U 1 1 5928D597
 P 7400 2100
@@
 $EndComp
 $Comp
-L CP C42
+L pocket_mixer-rescue:CP C42
 U 1 1 5928D59E
 P 7400 2900
@@
 NoConn ~ 1250 2600
 $Comp
-L GND #PWR095
+L pocket_mixer-rescue:GND #PWR095
 U 1 1 59375A2F
 P 3000 2400
@@
 $EndComp
 $Comp
-L GND #PWR096
+L pocket_mixer-rescue:GND #PWR096
 U 1 1 59375CE1
 P 2650 4050
@@
 $EndComp
 $Comp
-L GND #PWR097
+L pocket_mixer-rescue:GND #PWR097
 U 1 1 593774B8
 P 3000 3200
@@
 $EndComp
 $Comp
-L -12V #PWR109
+L pocket_mixer-rescue:-12V #PWR109
 U 1 1 5941CC23
 P 3550 1700
@@
 $EndComp
 $Comp
-L +12V #PWR098
+L pocket_mixer-rescue:+12V #PWR098
 U 1 1 5941CCFA
 P 3550 2300
@@
 $EndComp
 $Comp
-L +12V #PWR099
+L pocket_mixer-rescue:+12V #PWR099
 U 1 1 5941CD71
 P 3550 2700
@@
 $EndComp
 $Comp
-L -12V #PWR112
+L pocket_mixer-rescue:-12V #PWR112
 U 1 1 5941CDE8
 P 3550 3300
@@
 $EndComp
 $Comp
-L -12V #PWR124
+L pocket_mixer-rescue:-12V #PWR124
 U 1 1 5941CEBF
 P 8300 1700
@@
 $EndComp
 $Comp
-L +12V #PWR0100
+L pocket_mixer-rescue:+12V #PWR0100
 U 1 1 5941CF36
 P 8300 2300
@@
 $EndComp
 $Comp
-L +12V #PWR0101
+L pocket_mixer-rescue:+12V #PWR0101
 U 1 1 5941CFAD
 P 8300 2700
@@
 $EndComp
 $Comp
-L -12V #PWR127
+L pocket_mixer-rescue:-12V #PWR127
 U 1 1 5941D024
 P 8300 3300
@@
 $EndComp
 $Comp
-L -12V #PWR113
+L pocket_mixer-rescue:-12V #PWR113
 U 1 1 59421163
 P 4300 1200
@@
 $EndComp
 $Comp
-L +12V #PWR0102
+L pocket_mixer-rescue:+12V #PWR0102
 U 1 1 594211DA
 P 4650 1200
@@
 $EndComp
 $Comp
-L -12V #PWR128
+L pocket_mixer-rescue:-12V #PWR128
 U 1 1 59421391
 P 9050 1200
@@
 $EndComp
 $Comp
-L +12V #PWR0103
+L pocket_mixer-rescue:+12V #PWR0103
 U 1 1 59421408
 P 9400 1200

Commit message: :rocket: 2.0.0
Parts:
- added unit 3 of U8
- added unit 3 of U9
- C35, C36, C41, C42: symbol pocket_mixer-rescue:CP -> Device:CP
- C37, C38, C39, C40, C43, C44, C45, C46: symbol pocket_mixer-rescue:C -> Device:C
- J6, J7: symbol pocket_mixer-rescue:PJ3410 -> stahllabs:PJ3410
- R53, R54, R55, R56, R57, R58, R59, R60, R61, R62, R63, R64: symbol pocket_mixer-rescue:R -> Device:R
- RV10, RV9: symbol pocket_mixer-rescue:POT_Dual -> Device:R_POT_Dual
- U8, U9: value 4580 -> NJM4580; symbol pocket_mixer-rescue:4558 -> Amplifier_Operational:NJM4580
Connections:
- wire segments 72 -> 108
