File: pan_send.sch (KiCad schematic (older format))
At the start: 22 parts

Commit message: update to kicad version 5, bug fix layout
Parts:
- R35, R36, R37, R38, R39, R40, R41, R42, R43, R44, R45, R46, R47, R48, R49, R50, R51, R52: symbol R -> pocket_mixer-rescue:R
- RV5, RV6, RV7, RV8: symbol POT_Dual -> pocket_mixer-rescue:POT_Dual
Changed lines of the file:
@@
-EESchema Schematic File Version 2
-LIBS:power
-LIBS:device
-LIBS:transistors
-LIBS:conn
-LIBS:linear
-LIBS:regul
-LIBS:74xx
-LIBS:cmos4000
-LIBS:adc-dac
-LIBS:memory
-LIBS:xilinx
-LIBS:microcontrollers
-LIBS:dsp
-LIBS:microchip
-LIBS:analog_switches
-LIBS:motorola
-LIBS:texas
-LIBS:intel
-LIBS:audio
-LIBS:interface
-LIBS:digital-audio
-LIBS:philips
-LIBS:display
-LIBS:cypress
-LIBS:siliconi
-LIBS:opto
-LIBS:atmel
-LIBS:contrib
-LIBS:valves
-LIBS:switches
-LIBS:stahllabs
+EESchema Schematic File Version 4
 LIBS:pocket_mixer-cache
-EELAYER 25 0
+EELAYER 26 0
 EELAYER END
 $Descr A4 11693 8268
@@
 1-LEFT
 $Comp
-L R R36
+L pocket_mixer-rescue:R R36
 U 1 1 591F78CA
 P 2950 1350
@@
 $EndComp
 $Comp
-L R R37
+L pocket_mixer-rescue:R R37
 U 1 1 591F790A
 P 2950 1700
@@
 $EndComp
 $Comp
-L POT_Dual RV5
+L pocket_mixer-rescue:POT_Dual RV5
 U 1 1 59232745
 P 2500 1450
@@
 $EndComp
 $Comp
-L GND #PWR072
+L pocket_mixer-rescue:GND #PWR072
 U 1 1 59232E10
 P 2200 1550
@@
 $EndComp
 $Comp
-L GND #PWR073
+L pocket_mixer-rescue:GND #PWR073
 U 1 1 59232E34
 P 2200 1050
@@
 $EndComp
 $Comp
-L R R35
+L pocket_mixer-rescue:R R35
 U 1 1 59232E7F
 P 2950 1200
@@
 $EndComp
 $Comp
-L R R38
+L pocket_mixer-rescue:R R38
 U 1 1 59232E9D
 P 2950 1850
@@
 2-LEFT
 $Comp
-L R R40
+L pocket_mixer-rescue:R R40
 U 1 1 59233B64
 P 2950 2300
@@
 $EndComp
 $Comp
-L R R41
+L pocket_mixer-rescue:R R41
 U 1 1 59233B6B
 P 2950 2650
@@
 $EndComp
 $Comp
-L POT_Dual RV6
+L pocket_mixer-rescue:POT_Dual RV6
 U 1 1 59233B72
 P 2500 2400
@@
 $EndComp
 $Comp
-L GND #PWR074
+L pocket_mixer-rescue:GND #PWR074
 U 1 1 59233B79
 P 2200 2500
@@
 $EndComp
 $Comp
-L GND #PWR075
+L pocket_mixer-rescue:GND #PWR075
 U 1 1 59233B7F
 P 2200 2000
@@
 $EndComp
 $Comp
-L R R39
+L pocket_mixer-rescue:R R39
 U 1 1 59233B85
 P 2950 2150
@@
 $EndComp
 $Comp
-L R R42
+L pocket_mixer-rescue:R R42
 U 1 1 59233B8C
 P 2950 2800
@@
 3-LEFT
 $Comp
-L R R44
+L pocket_mixer-rescue:R R44
 U 1 1 592352BF
 P 2950 3250
@@
 $EndComp
 $Comp
-L R R45
+L pocket_mixer-rescue:R R45
 U 1 1 592352C5
 P 2950 3600
@@
 $EndComp
 $Comp
-L POT_Dual RV7
+L pocket_mixer-rescue:POT_Dual RV7
 U 1 1 592352CB
 P 2500 3350
@@
 $EndComp
 $Comp
-L GND #PWR076
+L pocket_mixer-rescue:GND #PWR076
 U 1 1 592352D1
 P 2200 3450
@@
 $EndComp
 $Comp
-L GND #PWR077
+L pocket_mixer-rescue:GND #PWR077
 U 1 1 592352D7
 P 2200 2950
@@
 $EndComp
 $Comp
-L R R43
+L pocket_mixer-rescue:R R43
 U 1 1 592352DD
 P 2950 3100
@@
 $EndComp
 $Comp
-L R R46
+L pocket_mixer-rescue:R R46
 U 1 1 592352E3
 P 2950 3750
@@
 4-LEFT
 $Comp
-L R R48
+L pocket_mixer-rescue:R R48
 U 1 1 592352F3
 P 2950 4200
@@
 $EndComp
 $Comp
-L R R49
+L pocket_mixer-rescue:R R49
 U 1 1 592352F9
 P 2950 4550
@@
 $EndComp
 $Comp
-L POT_Dual RV8
+L pocket_mixer-rescue:POT_Dual RV8
 U 1 1 592352FF
 P 2500 4300
@@
 $EndComp
 $Comp
-L GND #PWR078
+L pocket_mixer-rescue:GND #PWR078
 U 1 1 59235305
 P 2200 4400
@@
 $EndComp
 $Comp
-L GND #PWR079
+L pocket_mixer-rescue:GND #PWR079
 U 1 1 5923530B
 P 2200 3900
@@
 $EndComp
 $Comp
-L R R47
+L pocket_mixer-rescue:R R47
 U 1 1 59235311
 P 2950 4050
@@
 $EndComp
 $Comp
-L R R50
+L pocket_mixer-rescue:R R50
 U 1 1 59235317
 P 2950 4700
@@
 RETURN-LEFT
 $Comp
-L R R51
+L pocket_mixer-rescue:R R51
 U 1 1 5923810E
 P 2950 5500
@@
 $EndComp
 $Comp
-L R R52
+L pocket_mixer-rescue:R R52
 U 1 1 592381CD
 P 2950 5700

Commit message: :rocket: 2.0.0
Parts:
- removed RV5, RV6, RV7, RV8: 50kA, stahllabs:PTV112-4, symbol pocket_mixer-rescue:POT_Dual
- added RV5, RV6, RV7, RV8: 50k A, stahllabs:RK14K12D0A18, symbol stahllabs:POT_Dual_Common_Gnd
- R35, R36, R37, R38, R39, R40, R41, R42, R43, R44, R45, R46, R47, R48, R49, R50, R51, R52: footprint Resistors_SMD:R_1206 -> Resistor_SMD:R_1206_3216Metric; symbol pocket_mixer-rescue:R -> Device:R
Connections:
- net 1-LEFT: now also RV5.5
- net 1-RIGHT: now also RV5.3
- net 2-LEFT: now also RV6.5
- net 2-RIGHT: now also RV6.3
- net 3-LEFT: now also RV7.5
- net 3-RIGHT: now also RV7.3
- net 4-LEFT: now also RV8.5
- net 4-RIGHT: now also RV8.3
- net GND: now also RV5.1, RV6.1, RV7.1, RV8.1
- net at R37.1: now also RV5.4
- net at R35.1: now also RV5.2
- net at R41.1: now also RV6.4
- net at R39.1: now also RV6.2
- net at R45.1: now also RV7.4
- net at R43.1: now also RV7.2
- net at R49.1: now also RV8.4
- net at R47.1: now also RV8.2
Other:
- note added: "PANORAMA"
- note added: "STEREO SEND"
- note added: "not implemented"
