File: power_supply.sch (KiCad schematic (older format))
At the start: 29 parts, among them J10 CONN_01X02, J11 CONN_01X02, J8 USB_OTG, J9 CONN_01X02, SW1 SW_SPDT, U10 MCP73831, U11 LT1930, U12 LT1931

Commit message: update to kicad version 5, bug fix layout
Parts:
- C49, C50, C51, C52, C53, C54, C55, C56: symbol C -> pocket_mixer-rescue:C
- D1, D4: symbol LED -> pocket_mixer-rescue:LED
- D2, D3: symbol D_Schottky -> pocket_mixer-rescue:D_Schottky
- J10, J11, J9: symbol CONN_01X02 -> pocket_mixer-rescue:CONN_01X02
- J8: symbol USB_OTG -> pocket_mixer-rescue:USB_OTG
- L1: symbol L -> pocket_mixer-rescue:L
- L2: symbol CLS62NP-100NC -> pocket_mixer-rescue:CLS62NP-100NC
- R65, R66, R67, R68, R69, R70, R71: symbol R -> pocket_mixer-rescue:R
- SW1: symbol SW_SPDT -> pocket_mixer-rescue:SW_SPDT
- U10: symbol MCP73831 -> pocket_mixer-rescue:MCP73831
- U11: symbol LT1930 -> pocket_mixer-rescue:LT1930
- U12: symbol LT1931 -> pocket_mixer-rescue:LT1931
Other:
- moved on the sheet: C50

Commit message: :rocket: 2.0.0
Parts:
- removed C51, C52, C54: 4.7uF, Capacitors_SMD:C_1206, symbol pocket_mixer-rescue:C
- removed C53: 10pF, Capacitors_SMD:C_1206, symbol pocket_mixer-rescue:C
- removed C55: 10uF, Capacitors_SMD:C_1206, symbol pocket_mixer-rescue:C
- removed C56: 1uF, Capacitors_SMD:C_1206, symbol pocket_mixer-rescue:C
- removed D2, D3: D_Schottky, Diodes_SMD:D_SOD-123, symbol pocket_mixer-rescue:D_Schottky
- removed J10: CONN_01X02, Pin_Headers:Pin_Header_Straight_1x02_Pitch2.54mm, symbol pocket_mixer-rescue:CONN_01X02
- removed J11: CONN_01X02, stahllabs:JST_PH_S2B-PH-SM4-TB_02x2.00mm_Angled, symbol pocket_mixer-rescue:CONN_01X02
- removed J8: USB_OTG, stahllabs:USB_Micro-B, symbol pocket_mixer-rescue:USB_OTG
- removed L1: 10uH, stahllabs:Inductor_CR43NP-100MC, symbol pocket_mixer-rescue:L
- removed L2: 10uH, stahllabs:CLS62NP-100NC, symbol pocket_mixer-rescue:CLS62NP-100NC
- removed R67: 113k, Resistors_SMD:R_1206, symbol pocket_mixer-rescue:R
- removed R68: 13k3, Resistors_SMD:R_1206, symbol pocket_mixer-rescue:R
- removed R69: 84k5, Resistors_SMD:R_1206, symbol pocket_mixer-rescue:R
- removed R70: 10k, Resistors_SMD:R_1206, symbol pocket_mixer-rescue:R
- removed U11: LT1930, TO_SOT_Packages_SMD:SOT-23-5_HandSoldering, symbol pocket_mixer-rescue:LT1930
- removed U12: LT1931, TO_SOT_Packages_SMD:SOT-23-5_HandSoldering, symbol pocket_mixer-rescue:LT1931
- added D2: BAT20JFILM, Diode_SMD:D_SOD-323, symbol Device:D_Schottky
- added J10, J11: CONN_01X02, Connector_PinHeader_2.54mm:PinHeader_1x02_P2.54mm_Vertical, symbol Connector_Generic:Conn_01x02
- added J8: USB_C_Receptacle_Power_Only, stahllabs:USB_C_Receptacle_CUI_Devices_UJC-HP-3-SMT-TR, symbol stahllabs:USB_C_Receptacle_Power_Only
- added Q1: ZXMP6A13FTA, Package_TO_SOT_SMD:SOT-23, symbol stahllabs:ZXMP6A13FTA
- added R67: 100k, Resistor_SMD:R_1206_3216Metric, symbol Device:R
- added U11: DC-DC-Boost-Converter-Positive-Negative-Dual-Outp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, stahllabs:DC-DC-Boost-Converter-Positive-Negative-Dual-Output-Power-Supply, symbol stahllabs:DC-DC-Boost-Converter-Positive-Negative-Dual-Output-Power-Supply
- C49, C50: footprint Capacitors_SMD:C_1206 -> Capacitor_SMD:C_1206_3216Metric; symbol pocket_mixer-rescue:C -> Device:C
- D1, D4: symbol pocket_mixer-rescue:LED -> Device:LED
- J9: value CONN_01X02 -> 5V; footprint Pin_Headers:Pin_Header_Straight_1x02_Pitch2.54mm -> Connector_PinHeader_2.54mm:PinHeader_1x02_P2.54mm_Vertical; symbol pocket_mixer-rescue:CONN_01X02 -> Connector_Generic:Conn_01x02
- R65: value 330 -> 1k; footprint Resistors_SMD:R_1206 -> Resistor_SMD:R_1206_3216Metric; symbol pocket_mixer-rescue:R -> Device:R
- R66, R71: footprint Resistors_SMD:R_1206 -> Resistor_SMD:R_1206_3216Metric; symbol pocket_mixer-rescue:R -> Device:R
- SW1: symbol pocket_mixer-rescue:SW_SPDT -> Switch:SW_SPDT
- U10: footprint TO_SOT_Packages_SMD:SOT-23-5_HandSoldering -> Package_TO_SOT_SMD:SOT-23-5; symbol pocket_mixer-rescue:MCP73831 -> stahllabs:MCP73831
Connections:
- net -12V: now also U11.5 (-Vo)
- net 12V: now also U11.3 (+Vo); no longer R71.1
- net 5V: now also D2.2 (A), J8.A9 (VBUS), J8.B9 (VBUS), Q1.1, R67.1
- net GND: now also J10.2 (Pin_2), J11.2 (Pin_2), J8.A12 (GND), J8.B12 (GND), R67.2, U11.2 (GND), U11.4 (GND)
- net Vbat: now also C50.1, U10.3 (VBAT), J10.1 (Pin_1), J11.1 (Pin_1), Q1.3
- net at SW1.2 (B): now also R71.1, U11.1 (Vin)
- net at SW1.1 (A): now also D2.1 (K), Q1.2
- now unconnected: SW1.3 (C)
- no-connect marks 0 -> 4
Other:
- note added: "Autoswitching Power"
- note added: "DC DC Step-up Boost\nConverter module"
- note added: "DC-DC Step-up boost converter module\nhttps://de.aliexpress.com/item/32789671683.html?spm=a2g0s.9042311.0.0.27424c4d2Mwcoo"
- note added: "LiPo charger circuit"
- note added: "Testpoint"
- moved on the sheet: C49, C50, R65, R66, R71, SW1, U10
