File: mixerli.kicad_pcb (KiCad board)
At the start: 2 copper layers, 126 x 108 mm, 160 parts, among them J1 PJ3410, J10 CONN_01X02, J11 CONN_01X02, J2 PJ3410, J3 PJ3410, J4 PJ3410, J5 PJ3410, J6 PJ3410, J7 PJ3410, J8 USB_C_Receptacle_Power_Only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

Commit message: holes, jst bat, ..
Parts:
- added H1: MountingHole_Pad, MountingHole:MountingHole_3mm_Pad, F.Cu at (18.0, 92.0)
- added H2: MountingHole_Pad, MountingHole:MountingHole_3mm_Pad, F.Cu at (18.0, 192.0)
- added H3: MountingHole_Pad, MountingHole:MountingHole_3mm_Pad, F.Cu at (136.0, 92.0)
- added H4: MountingHole_Pad, MountingHole:MountingHole_3mm_Pad, F.Cu at (136.0, 192.0)
- J1, J2, J3, J4, J5, J6, J7: value PJ3410 -> QingPu_WQP-PJ366ST; footprint stahllabs:PJ3410 -> stahllabs:Jack_3.5mm_QingPu_WQP-PJ366ST_Vertical
- J10: footprint Connector_PinHeader_2.54mm:PinHeader_1x02_P2.54mm_Vertical -> Connector_JST:JST_PH_S2B-PH-K_1x02_P2.00mm_Horizontal
- J8: value USB_C_Receptacle_Power_Only -> UJC-HP-3-SMT-TR
- moved C48 3.29 mm to (111.5, 123.7)
- moved J11 2.62 mm to (66.4, 89.8), turned to 180 degrees
- moved J10 1.13 mm to (71.3, 91.3), turned to -90 degrees
- moved D1 1.09 mm to (23.9, 90.4)
- turned J1 to 0 degrees
- turned J2 to 0 degrees
- turned J3 to 0 degrees
- turned J4 to 0 degrees
- turned J5 to 0 degrees
- turned J6 to 0 degrees
- turned J7 to 0 degrees
Connections:
- net /Pan/Send/1-LEFT renamed /Input 1/LEFT
- net /Pan/Send/1-RIGHT renamed /Input 1/RIGHT
- net /Pan/Send/2-LEFT renamed /Input 2/LEFT
- net /Pan/Send/2-RIGHT renamed /Input 2/RIGHT
- net /Pan/Send/3-LEFT renamed /Input 3/LEFT
- net /Pan/Send/3-RIGHT renamed /Input 3/RIGHT
- net /Pan/Send/4-LEFT renamed /Input 4/LEFT
- net /Pan/Send/4-RIGHT renamed /Input 4/RIGHT
- net /Pan/Send/RETURN-RIGHT renamed /Input 5/RIGHT
- J8 pad A5: (no net) -> unconnected-(J8-PadA5)
- J8 pad B5: (no net) -> unconnected-(J8-PadB5)
- J8 pad S1: Net-(J8-PadS1) -> unconnected-(J8-PadS1)
- JP1 pad 1: Net-(J3-Pad3) -> Net-(J3-PadT)
- JP1 pad 2: Net-(J3-Pad2) -> Net-(J3-PadR)
- JP2 pad 1: Net-(J4-Pad3) -> Net-(J4-PadT)
- JP2 pad 2: Net-(J4-Pad2) -> Net-(J4-PadR)
- JP3 pad 1: Net-(J5-Pad3) -> Net-(J5-PadT)
- JP3 pad 2: Net-(J5-Pad2) -> Net-(J5-PadR)
- JP4 pad 1: Net-(J6-Pad3) -> Net-(J6-PadT)
- JP4 pad 2: Net-(J6-Pad2) -> Net-(J6-PadR)
- JP5 pad 1: Net-(J7-Pad3) -> Net-(J7-PadT)
- JP5 pad 2: Net-(J7-Pad2) -> Net-(J7-PadR)
- RV10 pad 3: Net-(J7-Pad2) -> Net-(J7-PadR)
- RV10 pad 6: Net-(J7-Pad3) -> Net-(J7-PadT)
- RV2 pad 3: Net-(J3-Pad2) -> Net-(J3-PadR)
- RV2 pad 6: Net-(J3-Pad3) -> Net-(J3-PadT)
- RV3 pad 3: Net-(J4-Pad2) -> Net-(J4-PadR)
- RV3 pad 6: Net-(J4-Pad3) -> Net-(J4-PadT)
- RV4 pad 3: Net-(J5-Pad2) -> Net-(J5-PadR)
- RV4 pad 6: Net-(J5-Pad3) -> Net-(J5-PadT)
- RV9 pad 3: Net-(J6-Pad2) -> Net-(J6-PadR)
- RV9 pad 6: Net-(J6-Pad3) -> Net-(J6-PadT)
- SW1 pad 3: (no net) -> unconnected-(SW1-Pad3)
Routing:
- net Net-(J5-PadT): track 0.00 -> 48.3 mm
- net Net-(J4-PadT): track 0.00 -> 48.0 mm
- net Net-(J3-PadT): track 0.00 -> 47.9 mm
- net Net-(J6-PadT): track 0.00 -> 47.9 mm
- net Net-(J3-Pad2): track 47.6 -> 0.00 mm
- net Net-(J6-Pad2): track 47.5 -> 0.00 mm
- net Net-(J5-Pad2): track 47.5 -> 0.00 mm
- net Net-(J4-Pad2): track 47.5 -> 0.00 mm
- net Net-(J7-Pad2): track 45.2 -> 0.00 mm
- net Net-(J7-PadT): track 0.00 -> 43.8 mm
- net Net-(J3-PadR): track 0.00 -> 40.7 mm
- net Net-(J6-PadR): track 0.00 -> 40.7 mm
- net Net-(J4-PadR): track 0.00 -> 40.7 mm
- net Net-(J5-PadR): track 0.00 -> 40.7 mm
- net Net-(J4-Pad3): track 38.5 -> 0.00 mm
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Other:
- board text added: "+12V"
- board text added: "-12V"
- board text added: "Gnd"
- board text added: "Vin"
- board text added: "mixerli"
- board text removed: "pocket mixer"

Commit message: mixerli 2.0.0 alpha
Parts:
- added G***: LOGO, stahllabs:LOGO_SGMK_Stamp_8.8mm, B.Cu at (93.3, 97.4)

Commit message: documentation / update kicad
Parts:
- moved C37 93.5 mm to (171.1, 100.7)
- moved C46 93.5 mm to (185.8, 96.7)
- moved C48 93.5 mm to (188.9, 71.3)
- moved C5 93.5 mm to (191.1, 75.6)
- moved G*** 93.5 mm to (170.6, 45.0)
- moved J10 93.5 mm to (148.6, 38.9)
- moved R47 93.5 mm to (159.0, 70.3)
- moved R48 93.5 mm to (171.1, 70.3)
- moved R54 93.5 mm to (157.1, 105.8)
- moved R58 93.5 mm to (157.1, 100.7)
- moved RV7 93.5 mm to (144.4, 63.6)
- moved RV8 93.5 mm to (164.4, 63.6)
- moved SW1 93.5 mm to (203.6, 38.0)
- moved U11 93.5 mm to (204.4, 121.3)
- moved C1 93.5 mm to (191.1, 89.3)
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
Commit message: gerber 2.0.0 final
Parts:
- added REF**: OSHW-Logo2_7.3x6mm_SilkScreen, Symbol:OSHW-Logo2_7.3x6mm_SilkScreen, B.Cu at (194.4, 44.1)
- J9: moved to B.Cu
- moved G*** 3.81 mm to (170.8, 41.1)
- moved J9 2.65 mm to (112.8, 50.7)
Routing:
- net /Power Supply/5V: track 53.2 -> 51.9 mm
Other:
- board text added: "+3.7V"
- board text added: "v2.0.0 github.com/stahlnow/mixerli"
- board text removed: "v2.0.0 alpha github.com/stahlnow/mixerli"
