File: fader.kicad_sch (KiCad schematic)
At the start: 18 parts, among them J7 PJ3410, U9 NJM4580

Commit message: holes, jst bat, ..
Parts:
- J3: renamed from J7; value PJ3410 -> QingPu_WQP-PJ366ST; footprint stahllabs:PJ3410 -> stahllabs:Jack_3.5mm_QingPu_WQP-PJ366ST_Vertical; symbol stahllabs:PJ3410 -> Connector:AudioJack3
- renumbered C41 to C17, C42 to C18, C43 to C21, C44 to C22, C45 to C25, C46 to C27, JP5 to JP1, R59 to R17, R60 to R18, R61 to R21, R62 to R22, R63 to R25, R64 to R26, RV10 to RV2, U9 to U5
Connections:
- net +12V: now also U5.8 (V+)
- net -12V: now also U5.4 (V-)
- net GND: now also J3.S; no longer J3.5 (sleeve)
- net LEFT: now also U5.7; no longer U5.1
- net at JP1.2 (B), RV2.3: now also J3.R; no longer J3.2 (ring)
- net at JP1.1 (A), RV2.6: now also J3.T; no longer J3.3 (tip)
- net at C18.2, R22.2: now also U5.5 (+); no longer U5.3 (+)
- net at C22.2, R18.1, R26.2: now also U5.6 (-); no longer U5.2 (-)
- no-connect marks 1 -> 0

Commit message: update LICENSE
Other:
- company: (none) -> stahllabs
- title: (none) -> mixerli

Commit message: v2.0.1: fixed pulldown resistors
Parts:
- J3: symbol Connector:AudioJack3 -> Connector_Audio:AudioJack3
Other:
- note added: "Note: Dual mono configuration The normally stereophonic input can be changed into a monophonic input where the signal is hardwired to both the left and the right channel resulting in a dual monophonic signal. This configuration requires two changes: - Ring pin of the jack must be removed - JP solder pad must be closed (soldered)"
- note removed: "Note: Dual mono configuration The normally stereophonic input can be changed into a monophonic input where the signal is hardwired to both the left and the right channel resulting in a dual monophonic signal. This change requires two changes: - Ring pin of the jack must be removed - JP solder pad must be closed (soldered)"
