File: mixerli.kicad_sch (KiCad schematic)
At the start: 41 parts, among them J1 PJ3410, J2 PJ3410, U1 NJM4580, U2 NJM4580, U3 NJM4580, U4 NJM4580

Commit message: holes, jst bat, ..
Parts:
- added H1, H2, H3, H4: MountingHole_Pad, MountingHole:MountingHole_3mm_Pad, symbol Mechanical:MountingHole_Pad
- J1, J2: value PJ3410 -> QingPu_WQP-PJ366ST; footprint stahllabs:PJ3410 -> stahllabs:Jack_3.5mm_QingPu_WQP-PJ366ST_Vertical; symbol stahllabs:PJ3410 -> Connector:AudioJack3
Connections:
- net GND: now also J1.S, J2.S; no longer J1.5 (sleeve), J2.5 (sleeve)
- net at C16.2, R16.2: now also J2.R; no longer J2.2 (ring)
- net at C9.2, R11.2: now also J1.T; no longer J1.3 (tip)
- net at C10.2, R12.2: now also J1.R; no longer J1.2 (ring)
- net at C15.2, R15.2: now also J2.T; no longer J2.3 (tip)
- no-connect marks 2 -> 0
Other:
- title: pocket mixer -> mixerli

Commit message: documentation / update kicad
Changed lines of the file:
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@@
   (title_block
     (title "mixerli")
-    (date "2022-04-07")
+    (date "2022-11-13")
     (rev "2.0.0a")
     (company "stahllabs")
+    (comment 1 "MIT License - Copyright (c) 2017 stahl")
+    (comment 2 "https://github.com/stahlnow/mixerli")
+    (comment 3 "level control slider and stereo rotary aux send level control.")
+    (comment 4 "LiPo powered 10 channel (4x2 + 1x2) stereo mixer featuring stereo input")
   )
   (junction (at 125.73 77.47) (diameter 0) (color 0 0 0 0)
@@
     (pin "1")
   )
-  (symbol (lib_id "Mechanical:MountingHole_Pad") (at 186.69 172.72 0) (unit 1)
+  (symbol (lib_id "Mechanical:MountingHole_Pad") (at 269.24 161.29 0) (unit 1)
     (in_bom yes) (on_board yes) (fields_autoplaced)
-    (property "Reference" "H2" (id 0) (at 189.23 170.6153 0)
+    (property "Reference" "H2" (id 0) (at 271.78 159.1853 0)
       (effects (font (size 1.27 1.27)) (justify left) hide)
     )
-    (property "Value" "MountingHole_Pad" (id 1) (at 189.23 171.8838 0)
+    (property "Value" "MountingHole_Pad" (id 1) (at 271.78 160.4538 0)
       (effects (font (size 1.27 1.27)) (justify left) hide)
     )
-    (property "Footprint" "MountingHole:MountingHole_3mm_Pad" (id 2) (at 186.69 172.72 0)
-      (effects (font (size 1.27 1.27)) hide)
-    )
-    (property "Datasheet" "~" (id 3) (at 186.69 172.72 0)
-      (effects (font (size 1.27 1.27)) hide)
-    )
-    (pin "1")
-  )
-  (symbol (lib_id "Mechanical:MountingHole_Pad") (at 191.77 172.72 0) (unit 1)
+    (property "Footprint" "MountingHole:MountingHole_3mm_Pad" (id 2) (at 269.24 161.29 0)
+      (effects (font (size 1.27 1.27)) hide)
+    )
+    (property "Datasheet" "~" (id 3) (at 269.24 161.29 0)
+      (effects (font (size 1.27 1.27)) hide)
+    )
+    (pin "1")
+  )
+  (symbol (lib_id "Mechanical:MountingHole_Pad") (at 274.32 161.29 0) (unit 1)
     (in_bom yes) (on_board yes) (fields_autoplaced)
-    (property "Reference" "H3" (id 0) (at 194.31 171.8838 0)
+    (property "Reference" "H3" (id 0) (at 276.86 160.4538 0)
       (effects (font (size 1.27 1.27)) (justify left) hide)
     )
-    (property "Value" "MountingHole_Pad" (id 1) (at 194.31 173.1522 0)
+    (property "Value" "MountingHole_Pad" (id 1) (at 276.86 161.7222 0)
       (effects (font (size 1.27 1.27)) (justify left) hide)
     )
-    (property "Footprint" "MountingHole:MountingHole_3mm_Pad" (id 2) (at 191.77 172.72 0)
-      (effects (font (size 1.27 1.27)) hide)
-    )
-    (property "Datasheet" "~" (id 3) (at 191.77 172.72 0)
-      (effects (font (size 1.27 1.27)) hide)
-    )
-    (pin "1")
-  )
-  (symbol (lib_id "Mechanical:MountingHole_Pad") (at 196.85 172.72 0) (unit 1)
+    (property "Footprint" "MountingHole:MountingHole_3mm_Pad" (id 2) (at 274.32 161.29 0)
+      (effects (font (size 1.27 1.27)) hide)
+    )
+    (property "Datasheet" "~" (id 3) (at 274.32 161.29 0)
+      (effects (font (size 1.27 1.27)) hide)
+    )
+    (pin "1")
+  )
+  (symbol (lib_id "Mechanical:MountingHole_Pad") (at 279.4 161.29 0) (unit 1)
     (in_bom yes) (on_board yes) (fields_autoplaced)
-    (property "Reference" "H4" (id 0) (at 199.39 170.6153 0)
+    (property "Reference" "H4" (id 0) (at 281.94 159.1853 0)
       (effects (font (size 1.27 1.27)) (justify left) hide)
     )
-    (property "Value" "MountingHole_Pad" (id 1) (at 199.39 171.8838 0)
+    (property "Value" "MountingHole_Pad" (id 1) (at 281.94 160.4538 0)
       (effects (font (size 1.27 1.27)) (justify left) hide)
     )
-    (property "Footprint" "MountingHole:MountingHole_3mm_Pad" (id 2) (at 196.85 172.72 0)
-      (effects (font (size 1.27 1.27)) hide)
-    )
-    (property "Datasheet" "~" (id 3) (at 196.85 172.72 0)
-      (effects (font (size 1.27 1.27)) hide)
-    )
-    (pin "1")
-  )
-  (symbol (lib_id "Mechanical:MountingHole_Pad") (at 181.61 172.72 0) (unit 1)
+    (property "Footprint" "MountingHole:MountingHole_3mm_Pad" (id 2) (at 279.4 161.29 0)
+      (effects (font (size 1.27 1.27)) hide)
+    )
+    (property "Datasheet" "~" (id 3) (at 279.4 161.29 0)
+      (effects (font (size 1.27 1.27)) hide)
+    )
+    (pin "1")
+  )
+  (symbol (lib_id "Mechanical:MountingHole_Pad") (at 264.16 161.29 0) (unit 1)
     (in_bom yes) (on_board yes) (fields_autoplaced)
-    (property "Reference" "H1" (id 0) (at 184.15 171.8838 0)
+    (property "Reference" "H1" (id 0) (at 266.7 160.4538 0)
       (effects (font (size 1.27 1.27)) (justify left) hide)
     )
-    (property "Value" "MountingHole_Pad" (id 1) (at 184.15 173.1522 0)
+    (property "Value" "MountingHole_Pad" (id 1) (at 266.7 161.7222 0)
       (effects (font (size 1.27 1.27)) (justify left) hide)
     )
-    (property "Footprint" "MountingHole:MountingHole_3mm_Pad" (id 2) (at 181.61 172.72 0)
-      (effects (font (size 1.27 1.27)) hide)
-    )
-    (property "Datasheet" "~" (id 3) (at 181.61 172.72 0)
+    (property "Footprint" "MountingHole:MountingHole_3mm_Pad" (id 2) (at 264.16 161.29 0)
+      (effects (font (size 1.27 1.27)) hide)
+    )
+    (property "Datasheet" "~" (id 3) (at 264.16 161.29 0)
       (effects (font (size 1.27 1.27)) hide)
     )
@@
       (reference "#PWR0122") (unit 1) (value "GND") (footprint "")
     )
+    (path "/00000000-0000-0000-0000-00005940313f/e6a5b190-be89-46cc-a14b-1fa03f35d78c"
+      (reference "#PWR?") (unit 1) (value "GND") (footprint "")
+    )
     (path "/00000000-0000-0000-0000-0000592a4f3f"

Commit message: update LICENSE
Other:
- note added: "Battery powered 10 channel (4x2 + 1x2) stereo mixer featuring stereo input level control slider and stereo rotary aux send level control."
- note removed: "LiPo powered 10 channel (4x2 + 1x2) stereo mixer featuring stereo input level control slider and stereo rotary aux send level control."

Commit message: v2.0.1: fixed pulldown resistors
Parts:
- J1, J2: symbol Connector:AudioJack3 -> Connector_Audio:AudioJack3
Connections:
- no-connect marks 0 -> 4
